File: couscous.kicad_sch (KiCad schematic)
At the start: 137 parts, among them SW1 SW_PUSH, SW10 SW_PUSH, SW11 SW_PUSH, SW12 SW_PUSH, SW13 SW_PUSH, SW14 SW_PUSH, SW15 SW_PUSH, SW16 SW_PUSH, SW17 SW_PUSH, SW18 SW_PUSH, SW19 SW_PUSH, SW2 SW_PUSH, SW20 SW_PUSH, SW21 SW_PUSH, SW22 SW_PUSH, SW23 SW_PUSH, SW24 SW_PUSH, SW25 SW_PUSH, SW26 SW_PUSH, SW27 SW_PUSH, SW28 SW_PUSH, SW29 SW_PUSH, SW3 SW_PUSH, SW30 SW_PUSH, SW31 SW_PUSH, SW32 SW_PUSH, SW33 SW_PUSH, SW34 SW_PUSH, SW35 SW_PUSH, SW36 SW_PUSH, SW37 SW_PUSH, SW38 SW_PUSH, SW39 SW_PUSH, SW4 SW_PUSH, SW40 SW_PUSH, SW41 SW_PUSH, SW42 SW_PUSH, SW43 SW_PUSH, SW44 SW_PUSH, SW45 SW_PUSH, SW46 SW_PUSH, SW47 SW_PUSH, SW48 SW_PUSH, SW49 SW_PUSH, SW5 SW_PUSH, SW50 SW_PUSH, SW51 SW_PUSH, SW52 SW_PUSH, SW53 SW_PUSH, SW54 SW_PUSH, SW55 SW_PUSH, SW56 SW_PUSH, SW57 SW_PUSH, SW58 SW_PUSH, SW59 SW_PUSH, SW6 SW_PUSH, SW60 SW_PUSH, SW61 SW_SPST, SW62 SW_SPST, SW63 SW_SPST, SW64 SW_SPST, SW65 SW_SPST, SW7 SW_PUSH, SW8 SW_PUSH, SW9 SW_PUSH, U1 SeeeduinoXIAO

Commit message: Placing
Parts:
- added D67, D68, D69, D70: LED_RGBW, qwelyt:LED_RGBW_SMD_5050, symbol qwelyt:LED_RGBW
Connections:
- net +5V is gone; now on net 5V: SW61.2 (B)
- net GND: now also U1.13 (GND), D70.1, D70.2, D70.3, D70.4; no longer D66.1, D66.2, D66.3, D66.4
- net 5V: now reaches U1.14 (5V)
- new net: D69.4, D70.5
- new net: D69.3, D70.6
- new net: D69.2, D70.7
- new net: D69.1, D70.8
- new net: D68.4, D69.5
- new net: D68.3, D69.6
- new net: D68.2, D69.7
- new net: D68.1, D69.8
- new net: D67.1, D68.8
- new net: D67.2, D68.7
- new net: D67.3, D68.6
- new net: D67.4, D68.5
- new net: D66.4, D67.5
- new net: D66.3, D67.6
- new net: D66.2, D67.7
- new net: D66.1, D67.8
- no-connect marks 0 -> 7

Commit message: Routing!
Connections:
- net Pin3: now reaches D25.1 (K), D26.2 (A), D27.1 (K), D28.2 (A), D29.1 (K), D30.2 (A), D31.1 (K), D32.2 (A), D33.1 (K), D34.2 (A), D35.1 (K), D36.2 (A)
- net Pin3: now also U1.3 (PA10_A2_D2); no longer U1.9 (PA7_A8_D8_SCK)
- net Pin8: now reaches SW17.1, SW18.1, SW29.1, SW30.1, SW41.1, SW42.1, SW5.1, SW53.1, SW54.1, SW6.1
- net Pin8: now also U1.8 (PB09_A7_D7_RX); no longer U1.3 (PA10_A2_D2)
- net Pin10: now reaches SW10.1, SW21.1, SW22.1, SW33.1, SW34.1, SW45.1, SW46.1, SW57.1, SW58.1, SW9.1
- net Pin10: now also U1.10 (PA5_A9_D9_MISO); no longer U1.5 (PA8_A4_D4_SDA)
- net Pin6: now reaches SW1.1, SW13.1, SW14.1, SW2.1, SW25.1, SW26.1, SW37.1, SW38.1, SW49.1, SW50.1
- net Pin6: now also U1.6 (PA9_A5_D5_SCL); no longer U1.1 (PA02_A0_D0)
- net Pin1: now reaches D49.1 (K), D50.2 (A), D51.1 (K), D52.2 (A), D53.1 (K), D54.2 (A), D55.1 (K), D56.2 (A), D57.1 (K), D58.2 (A), D59.1 (K), D60.2 (A)
- net Pin1: now also U1.1 (PA02_A0_D0); no longer U1.11 (PA6_A10_D10_MOSI)
- net Pin9: now reaches SW19.1, SW20.1, SW31.1, SW32.1, SW43.1, SW44.1, SW55.1, SW56.1, SW7.1, SW8.1
- net Pin9: now also U1.9 (PA7_A8_D8_SCK); no longer U1.4 (PA11_A3_D3)
- net Pin5: now reaches D1.1 (K), D10.2 (A), D11.1 (K), D12.2 (A), D2.2 (A), D3.1 (K), D4.2 (A), D5.1 (K), D6.2 (A), D7.1 (K), D8.2 (A), D9.1 (K)
- net Pin5: now also U1.5 (PA8_A4_D4_SDA); no longer U1.7 (PB08_A6_D6_TX)
- net Pin2: now reaches D37.1 (K), D38.2 (A), D39.1 (K), D40.2 (A), D41.1 (K), D42.2 (A), D43.1 (K), D44.2 (A), D45.1 (K), D46.2 (A), D47.1 (K), D48.2 (A)
- net Pin2: now also U1.2 (PA4_A1_D1); no longer U1.10 (PA5_A9_D9_MISO)
- net Pin7: now reaches SW15.1, SW16.1, SW27.1, SW28.1, SW3.1, SW39.1, SW4.1, SW40.1, SW51.1, SW52.1
- net Pin7: now also U1.7 (PB08_A6_D6_TX); no longer U1.2 (PA4_A1_D1)
- net Pin4: now reaches D13.1 (K), D14.2 (A), D15.1 (K), D16.2 (A), D17.1 (K), D18.2 (A), D19.1 (K), D20.2 (A), D21.1 (K), D22.2 (A), D23.1 (K), D24.2 (A)
- net Pin4: now also U1.4 (PA11_A3_D3); no longer U1.8 (PB09_A7_D7_RX)
- net Pin11: now reaches SW11.1, SW12.1, SW23.1, SW24.1, SW35.1, SW36.1, SW47.1, SW48.1, SW59.1, SW60.1
- net Pin11: now also U1.11 (PA6_A10_D10_MOSI); no longer U1.6 (PA9_A5_D5_SCL)

Commit message: Route everything
Everything should be routed now.
Parts:
- removed D67, D68, D69, D70: LED_RGBW, qwelyt:LED_RGBW_SMD_5050, symbol qwelyt:LED_RGBW
- added R10, R11, R13, R14, R15, R17, R18, R19, R21, R22, R23, R25, R26, R27, R29, R6, R7, R9: 9Ω, Resistor_SMD:R_0603_1608Metric_Pad0.98x0.95mm_HandSolder, symbol Device:R
- added R12, R16, R20, R24, R28, R8: 15Ω, Resistor_SMD:R_0603_1608Metric_Pad0.98x0.95mm_HandSolder, symbol Device:R
Connections:
- net GND: now also D61.1, D61.2, D61.3, D61.4, D62.1, D62.2, D62.3, D62.4, D63.1, D63.2, D63.3, D63.4, D64.1, D64.2, D64.3, D64.4, D65.1, D65.2, D65.3, D65.4, D66.1, D66.2, D66.3, D66.4
- net at D63.8: now also R14.1; no longer D62.1
- net at D63.7: now also R15.1; no longer D62.2
- net at D63.6: now also R16.1; no longer D62.3
- net at D63.5: now also R17.1; no longer D62.4
- net at D62.5: now also R13.1; no longer D61.4
- net at D62.6: now also R12.1; no longer D61.3
- net at D62.7: now also R11.1; no longer D61.2
- net at D62.8: now also R10.1; no longer D61.1
- net at R3.2: now also R12.2, R16.2, R20.2, R24.2, R28.2, R8.2; no longer D61.6
- net at D64.8: now also R18.1; no longer D63.1
- net at D64.7: now also R19.1; no longer D63.2
- net at D64.6: now also R20.1; no longer D63.3
- net at D64.5: now also R21.1; no longer D63.4
- net at R5.2: now also R10.2, R14.2, R18.2, R22.2, R26.2, R6.2; no longer D61.8
- net at D66.8: now also R26.1; no longer D65.1
- net at D66.7: now also R27.1; no longer D65.2
- net at D66.6: now also R28.1; no longer D65.3
- net at D66.5: now also R29.1; no longer D65.4
- net at D65.5: now also R25.1; no longer D64.4
- net at D65.6: now also R24.1; no longer D64.3
- net at D65.7: now also R23.1; no longer D64.2
- net at D65.8: now also R22.1; no longer D64.1
- net at R2.2: now also R13.2, R17.2, R21.2, R25.2, R29.2, R9.2; no longer D61.5
- net at R4.2: now also R11.2, R15.2, R19.2, R23.2, R27.2, R7.2; no longer D61.7
- new net: D61.6, R8.1
- new net: D61.8, R6.1
- new net: D61.5, R9.1
- new net: D61.7, R7.1
Other:
- moved on the sheet: D1, D10, D11, D12, D13, D14, D15, D16, D17, D18, D19, D2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

Commit message: Update pcb
Parts:
- renumbered D61 to LED1, D62 to LED2, D63 to LED3, D64 to LED4, D66 to LED5, D65 to LED6
Connections:
- net at R23.1: now also LED5.7; no longer LED6.7
- net at R24.1: now also LED5.6; no longer LED6.6
- net at R29.1: now also LED6.5; no longer LED5.5
- net at R25.1: now also LED5.5; no longer LED6.5
- net at R28.1: now also LED6.6; no longer LED5.6
- net at LED6.8: now also R26.1; no longer R22.1
- net at R27.1: now also LED6.7; no longer LED5.7
- net at LED5.8: now also R22.1; no longer R26.1
Other:
- moved on the sheet: LED5, LED6
